Commit message: Update generated files

File: lmtclam/ikfast/_gen_clam.urdf (robot description, URDF)
Before this commit: robot lmtclam, 15 links, 14 joints
Links:
- removed link gripper_finger_link
- removed link l_gripper_fwd_link
- removed link l_gripper_pincher_link
- removed link r_gripper_aft_link
- removed link r_gripper_fwd_link
- removed link r_gripper_pincher_link
- link arm_base_link: geometry collision mesh filename=package://lmtclam/model/stl/base_link_simple.STL scale=0.001 0.001 0.001; visual mesh filename=package://lmtclam/model/stl/base_link.STL scale=0.001 0.001 0.001
- link elbow_pitch_link: geometry collision mesh filename=package://lmtclam/model/stl/elbow_pitch_link_simple.STL scale=0.001 0.001 0.001; visual mesh filename=package://lmtclam/model/stl/elbow_pitch_link.STL scale=0.001 0.001 0.001
- link elbow_roll_link: geometry collision mesh filename=package://lmtclam/model/stl/elbow_roll_link_simple.STL scale=0.001 0.001 0.001; visual mesh filename=package://lmtclam/model/stl/elbow_roll_link.STL scale=0.001 0.001 0.001
- link gripper_roll_link: mass 1.0 -> None; geometry 
- link shoulder_pan_link: geometry collision mesh filename=package://lmtclam/model/stl/shoulder_pan_link_simple.STL scale=0.001 0.001 0.001; visual mesh filename=package://lmtclam/model/stl/shoulder_pan_link.STL scale=0.001 0.001 0.001
- link shoulder_pitch_link: geometry collision mesh filename=package://lmtclam/model/stl/shoulder_pitch_link_simple.STL scale=0.001 0.001 0.001; visual mesh filename=package://lmtclam/model/stl/shoulder_pitch_link.STL scale=0.001 0.001 0.001
- link wrist_pitch_link: geometry collision box size=0.0506 .0356 0.041; collision box size=0.0506 .0356 0.041
- link wrist_roll_link: geometry collision mesh filename=package://lmtclam/model/stl/wrist_roll_link_simple.STL scale=0.001 0.001 0.001; visual mesh filename=package://lmtclam/model/stl/wrist_roll_link.STL scale=0.001 0.001 0.001
Joints:
- removed joint gripper_finger_joint
- removed joint gripper_finger_pincher_joint
- removed joint l_gripper_fwd_joint
- removed joint r_gripper_aft_joint
- removed joint r_gripper_aft_pincher_joint
- removed joint r_gripper_fwd_joint
